File: hw-rt5350F_proto-r01/prj-kicad/fma-brick-r01.kicad_pcb (KiCad board)
At the start: 2 copper layers, 80 x 90 mm, 32 parts, among them J1 CONN_DC10A-2.1, J2 CONN_RJ45-L, J3 CONN_RJ45-L, J4 CONN_RJ45-L, P1 JUMPER, T100 TRANSFORMER_1:1, T200 TRANSFORMER_1:1, T300 TRANSFORMER_1:1, U1 LM2596

Commit message: = UPD: Design of rev0.1 is complete and ready for verify
Parts:
- added C10: 1uF, SMD0603, F.Cu at (149.3, 129.2)
- added C6: 1uF, SMD0603, F.Cu at (116.3, 134.7)
- added C7: 1uF, SMD0603, F.Cu at (176.4, 126.6)
- added C8: 1uF, SMD0603, F.Cu at (122.7, 124.1)
- added C9: 47uF, C_TAJB, F.Cu at (119.5, 125.6)
- added J5: CONN_4, CONN_4, F.Cu at (177.2, 132.6)
- added J6: CONN_USB_A, CONN_61400416021, F.Cu at (128.1, 129.7)
- added L201: FB100, SMD0603, F.Cu at (141.1, 74.1)
- added L301: FB100, SMD0603, F.Cu at (161.2, 74.1)
- added R203: 49.9, SMD0603, F.Cu at (144.6, 79.6)
- added R204: 49.9, SMD0603, F.Cu at (146.1, 81.1)
- added R205: 49.9, SMD0603, F.Cu at (150.9, 81.1)
- added R206: 49.9, SMD0603, F.Cu at (152.4, 79.6)
- added TP1: CONN_1, TP_PIN, F.Cu at (148.6, 127.0)
- added TP2: CONN_1, TP_PIN, F.Cu at (146.1, 127.0)
- added TP3: CONN_1, TP_PIN, F.Cu at (143.5, 127.0)
- added TP4: CONN_1, TP_PIN, F.Cu at (141.0, 127.0)
- added TP5: CONN_1, TP_PIN, F.Cu at (138.4, 127.0)
- added TP6: CONN_1, TP_PIN, F.Cu at (135.9, 127.0)
- added U2: CONN_USD, CONN_114-00841-68, F.Cu at (107.8, 130.1)
- added fma_logo: VAL**, fma_logo, F.Cu at (156.7, 136.2)
- added ohw_logo: VAL**, ohw_logo, F.Cu at (101.3, 110.4)
- J1: footprint CONN_DC-10 -> CONN_DC-694106106102
- moved C102 2.86 mm to (133.4, 76.6), turned to 270 degrees
- moved J1 2.51 mm to (108.0, 55.0), turned to 0 degrees
- moved R301 1.92 mm to (176.0, 70.8), turned to 270 degrees
- moved R302 1.06 mm to (161.2, 70.8), turned to 90 degrees
- moved J4 0.91 mm to (168.6, 57.9)
- moved C302 0.69 mm to (176.0, 76.6)
- moved C301 0.54 mm to (161.2, 76.6)
Connections:
- MOD1 pad 1: N-0000012 -> +3.3V
- MOD1 pad 23: N-0000083 (its old number) -> UART_TX
- MOD1 pad 25: N-0000079 (its old number) -> UART_RX
- MOD1 pad 30: N-0000073 (its old number) -> USB_DM
- MOD1 pad 32: N-0000082 (its old number) -> USB_DP
- MOD1 pad 51: N-0000072 (its old number) -> SPI_CS
- MOD1 pad 54: N-000007 (its old number) -> +3.3V
- MOD1 pad 57: N-0000013 -> SPI_MISO
- MOD1 pad 58: N-0000025 (its old number) -> SPI_MOSI
- MOD1 pad 59: N-0000024 (its old number) -> SPI_CLK
- MOD1 pad 6: N-0000094 (its old number) -> JTAG_TDI
- MOD1 pad 7: N-0000093 -> JTAG_TMS
- MOD1 pad 8: N-0000092 -> JTAG_TCK
- MOD1 pad 9: N-0000091 (its old number) -> JTAG_TDO
Routing:
- net GND: track 200.6 -> 719.6 mm, vias 20 -> 92
- net +3.3V: track 0.00 -> 150.1 mm, vias 0 -> 1
- net SPI_CS: track 0.00 -> 83.9 mm, vias 0 -> 1
- net +1.8V: track 0.00 -> 64.9 mm, vias 0 -> 1
- net SPI_MISO: track 0.00 -> 49.2 mm
- net SPI_MOSI: track 0.00 -> 47.8 mm
- net SPI_CLK: track 0.00 -> 43.7 mm
- net USB_DP: track 0.00 -> 43.1 mm
- net USB_DM: track 0.00 -> 41.3 mm, vias 0 -> 1
- net +5V: track 56.0 -> 85.1 mm, vias 0 -> 2
- net UART_TX: track 0.00 -> 21.8 mm
- net RX0_N: track 0.00 -> 19.9 mm, vias 0 -> 2
- net UART_RX: track 0.00 -> 17.5 mm
- net RX3_N: track 0.00 -> 16.1 mm, vias 0 -> 2
- net RX0_P: track 0.00 -> 16.1 mm, vias 0 -> 2
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- added copper zone on B.Cu, net GND
Other:
- board text added: "Agilack 2015 CC-by-SA"
- board text added: "FMA-Brick r0.1"
