File: hw-rt5350F_proto-r01/prj-kicad/fma-brick-r01.sch (KiCad schematic (older format))
At the start: 32 parts, among them J1 CONN_DC10A-2.1, J2 CONN_RJ45-L, J3 CONN_RJ45-L, J4 CONN_RJ45-L, P1 JUMPER, T100 TRANSFORMER_1:1, T200 TRANSFORMER_1:1, T300 TRANSFORMER_1:1, U1 LM2596

Commit message: = UPD: Design of rev0.1 is complete and ready for verify
Parts:
- added C10, C6, C7, C8: 1uF, symbol C
- added C9: 47uF, symbol CP
- added J5: CONN_4, symbol CONN_4
- added J6: CONN_USB_A, symbol CONN_USB_A
- added L201, L301: FB100, symbol INDUCTOR
- added R203, R204, R205, R206: 49.9, symbol R
- added TP1, TP2, TP3, TP4, TP5, TP6: CONN_1, symbol CONN_1
- added U2: CONN_USD, symbol CONN_USD
Connections:
- net labels added: +3.3V, JTAG_TCK, JTAG_TDI, JTAG_TDO, JTAG_TMS, SPI_CLK, SPI_CS, SPI_MISO, SPI_MOSI, UART_RX, UART_TX, USB_DM, USB_DP
- wire segments 155 -> 239
- no-connect marks 15 -> 39
Other:
- moved on the sheet: C201, MOD1A, MOD1C
